Commit message: add camera plugin

File: tm_grasp_description/urdf/robot_hand_gazebo_plugin.urdf (robot description, URDF)
Before this commit: robot tm700, 22 links, 21 joints
Links:
- added link camera_link
- added link camera_link_optical
Joints:
- added joint camera_joint: type fixed, parent tip_link, child camera_link, origin xyz=0 0.08 0.0421 rpy=0 0 0
- added joint camera_optical_joint: type fixed, parent camera_link, child camera_link_optical, origin xyz=0 0 0 rpy=-1.57079632679 0 -1.57079632679

Commit message: fix the camera position bug

File: tm_grasp_description/urdf/robot_hand_gazebo_plugin.urdf (robot description, URDF)
Before this commit: robot tm700, 24 links, 23 joints
Joints:
- joint camera_joint: origin xyz=0 0.08 0.0421 rpy=0 0 0 -> xyz=0.02 0.08 0.05 rpy=0 0 0
- joint camera_optical_joint: origin xyz=0 0 0 rpy=-1.57079632679 0 -1.57079632679 -> xyz=0 0 0 rpy=-1.57079632679 -1.57079632679 0
